File: pecanpico8.kicad_pcb (KiCad board)
At the start: 4 copper layers, 29.8 x 33.7 mm, 153 parts, among them IC1 SPV1040, IC2 TPS62260, IC3 ADP322ACPZ-115-R7, IC4 Si4464, IC5 STM32F745IGKx, IC6 EVA-7M, IC7 PAC1720, IC8 BME280, P1 CONN_01X25, P2 CONN_01X11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

Commit message: Increased via dia, moved drillings in panel
Routing:
- net +3V3: track 36.4 -> 35.1 mm
- net GND: track 118.0 -> 117.5 mm, vias 134 -> 131
- net +SOL: track 50.6 -> 50.2 mm, vias 6 -> 5
- net +1V8: track 151.4 -> 151.7 mm, vias 33 -> 32
Other:
- net class Default: clearance 0.15 -> 0.1; via_dia 0.3 -> 0.4
- rule trace_clearance: 0.15 -> 0.1
- rule via_min_size: 0.3 -> 0.4
