File: hardware/pecanpico8.sch (KiCad schematic (older format))
At the start: 148 parts, among them IC1 SPV1040, IC2 TPS62260, IC3 ADP322ACPZ-115-R7, IC4 Si4464, IC5 STM32F745IGKx, IC6 EVA-7M, IC7 PAC1720, IC8 BME280, P1 CONN_01X25, P2 CONN_01X11, P3 USB_OTG, P4 SMA Edge, P5 CONN_01X02, Q1 FDN306P, X1 KT2016K26000BCW18ZAS

Commit message: Started developement of rev 8b Changed USB Connector: Mini => Micro Connected CAM_EN to STM32 Added battery jumper switch at programming header Added solar input at programmer header Removed LED outputs at programmer header Removed Testpads at BOOT0 Moved parts around
Parts:
- removed D10: red, stm32f7:LED_0603, symbol LED
- removed D11: yellow, stm32f7:LED_0603, symbol LED
- removed R34: 1k5, stm32f7:R_0603, symbol R
- removed R37: 330R, stm32f7:R_0603, symbol R
- removed W1: TEST, stm32f7:R_0402, symbol TEST
- P3: footprint Connect:USB_Mini-B -> stm32f7:USB_Micro-B
Connections:
- net +1V8: now also P5.2 (P2); no longer P2.1 (P1)
- net +BATT: now also P2.11 (P11); no longer W11.1
- net +SOL: now also P2.9 (P9)
- net CAM_EN: now also IC5.K1 (PF7/ADC3_IN5/QUADSPI_BK1_IO2/SAI1_MCLK_B/SPI5_SCK/TIM11_CH1/UART7_TX)
- net GND: now also P2.2 (P2), P2.8 (P8); no longer P2.11 (P11), P2.3 (P3), P5.2 (P2)
- net IO_LED1: no longer P2.7 (P7)
- net IO_LED2: no longer P2.8 (P8)
- net IO_RXD: now also P2.7 (P7); no longer P2.10 (P10)
- net IO_TXD: now also P2.6 (P6); no longer P2.9 (P9)
- net SWD_NRST: now also P2.4 (P4); no longer P2.5 (P5)
- net SWD_SWCLK: now also P2.1 (P1); no longer P2.2 (P2)
- net SWD_SWDIO: now also P2.3 (P3); no longer P2.4 (P4)
- net SWD_SWO: now also P2.5 (P5); no longer P2.6 (P6)
- net USB_VUSB: now reaches IC5.E15 (DAC_EXTI9/DCMI_D0/I2C3_SMBA/I2S2_CK/SPI2_SCK/TIM1_CH2/USART1_TX/USB_OTG_FS_VBUS/PA9)
- net USB_VUSB: now also F1.2, P3.1 (VCC), R33.1
- new net BATT_CONN: P2.10 (P10), W11.1
Other:
- moved on the sheet: D8, D9, F1, P3

Commit message: GPS
- GPS Antenna went to the backside, so save space.
- We also use IPEX connectors for the GPS Antenna instead but you can also solder a wire on the connector pad instead.

Transmitter

- The space which I won, went into the LPF of the transceiver.
- We use an LFCN LPF by Mini-Circuits. They are more expensive (~US$5) but work perfectly for us.
- We also added a RX/TX switch to it. I did this because an Australian friend found out how to receive AFSK APRS with the Si4464.
- The transmitter also got that fancy IPEX connector for which you can find prebuild 70cm wire-antennas on Ebay for US$1.

Camera

- I discarded the FFC connector and replaced it with a custom 50mil edge-header (on which you can attach a standard 50mil header)
- But we planned to use cameras like these: https://sc02.alicdn.com/kf/HTB1PjEGKVXXXXaYXXXXq6xXFXXX1/2-0-Mega-Pixels-CMOS-OV2640-camera.jpg
- They are soldered on a separate daughter board. That daughter board is directly soldered to the edge of the Pecan. The dautherboard is then looking downwards
- There can be soldered a separated BME280 on the daughterboard too but that's optional

Connectors
- The side connector has a different Pinout. the first 2 pins connect the battery to the circuit itself. By removing a jumper on the header, you may disconnect the battery from the circuit.
- On the bottom you have a BOOT0. That pin got an additional pulldown, so the tracker doesn't fall accidentally into the bootloader.

USB
- I replaced the Mini USB connector with a Micro USB connector while you need much force to remove plug.
- I also connected the USB port to another specific pin on the STM32. While VUSB wasn't connected, USB wouldn't startup unfortunately.
- Connected USB to PB port instead of port PA
Parts:
- removed C25, C27: 22p, stm32f7:C_0402, symbol C
- removed C26: 1p8, stm32f7:C_0402, symbol C
- removed L5, L6: 68n, stm32f7:R_0603, symbol INDUCTOR
- removed P1: CONN_01X25, stm32f7:FFC1x24_0.5mm, symbol CONN_01X25
- removed W2, W5: Pad, stm32f7:PAD_6x1.5, symbol TEST_1P
- removed W25: Pad, Measurement_Points:Measurement_Point_Round-SMD-Pad_Small, symbol TEST_1P
- removed W4: Pad, stm32f7:PAD_4x4, symbol TEST_1P
- added D10: red, stm32f7:LED_0603, symbol LED
- added IC9: BME280, stm32f7:BME280, symbol BME280
- added P1: CONN_02X13, stm32f7:OV2640_Header, symbol CONN_02X13
- added P6: IPX 2mm, stm32f7:IPX_2mm, symbol Coax_connector
- added P7: CONN_02X13, stm32f7:OV2640_Socket, symbol CONN_02X13
- added R34, R37, R38: 0R, stm32f7:R_0402, symbol R
- added U1: AS-213, stm32f7:SC-70-6, symbol RF_SWITCH
- added U2: LFCN-120, stm32f7:FV1206, symbol LPF
- added U3: uctronics OV2640, stm32f7:OV2640, symbol uctronics_OV2640
- added W1: Testpad, stm32f7:Testpad, symbol TEST_1P
- C17: value NA -> 100n
- C21: value 18p -> 100n
- C24: value 4p7 -> 470p
- P4: value SMA Edge -> IPX 2mm; footprint stm32f7:SMA_EDGE -> stm32f7:IPX_2mm
- R1: value 22k -> 220k
- R2: value 10k -> 100k
- R27: value NA -> 0R
- R31: value NA -> 100k
- W12, W13, W14, W15, W16, W17, W18, W19, W20, W21, W22, W23, W24, W26, W27: footprint Measurement_Points:Measurement_Point_Round-SMD-Pad_Small -> stm32f7:Testpad
- W3: value Pad -> Testpad; footprint stm32f7:PAD_3x1.5 -> stm32f7:Testpad
Connections:
- net +1V35: now also P1.7 (P7), P1.9 (P9)
- net +1V8: now also C17.1, IC9.2 (CSB), IC9.6 (VDDIO), IC9.8 (VDD), P1.3 (P3), P7.3 (P3), R34.1; no longer IC6.20 (VCC_IO), R31.1
- net +3V3: now also R38.1
- net BOOT0: now also R31.1
- net CAM_D2: now also P1.19 (P19)
- net CAM_D3: now also P1.24 (P24)
- net CAM_D4: now also P1.23 (P23)
- net CAM_D5: now also P1.22 (P22)
- net CAM_D6: now also P1.4 (P4)
- net CAM_D7: now also P1.17 (P17)
- net CAM_D8: now also P1.10 (P10)
- net CAM_D9: now also P1.18 (P18)
- net CAM_HREF: now also P1.11 (P11)
- net CAM_PCLK: now also P1.20 (P20)
- net CAM_RESET: now also P1.6 (P6)
- net CAM_VSYNC: now also P1.16 (P16)
- net CAM_XCLK: now also P1.21 (P21)
- net CLOCK_26M: no longer C17.1
- net GND: now also C17.2, IC5.P12 (CAN2_RX/ETH_TXD0/I2C2_SMBA/I2S2_WS/SPI2_NSS/TIM1_BKIN/USART3_CK/USB_OTG_HS_ID/USB_OTG_HS_ULPI_D5/PB12), R31.2, IC9.1 (GND), IC9.5 (SDO), IC9.7 (GND), P1.1 (P1), P1.2 (P2), P1.25 (P25), P1.26 (P26), P6.2, P7.1 (P1), P7.2 (P2), P7.25 (P25), P7.26 (P26), U1.2 (GND), U2.3 (GND), U3.11 (DGND), U3.16 (AGND), U3.18 (DGND), U3.6 (DGND)
- net GPS_IRQ: now also IC5.B15 (CAN1_TX/SAI2_FS_B/TIM1_ETR/USART1_RTS/USB_OTG_FS_DP/PA12); no longer IC5.B14 (DCMI_D8/I2S3_CK/QUADSPI_BK1_IO1/SDMMC1_D2/SPI3_SCK/UART4_TX/USART3_TX/PC10)
- net I2C_SCL: now also P1.14 (P14)
- net I2C_SDA: now also P1.12 (P12)
- net PAC_ALERT: now also IC5.N13 (FMC_A17/FMC_ALE/I2C4_SCL/LPTIM1_IN1/QUADSPI_BK1_IO1/SAI2_FS_A/TIM4_CH1/USART3_RTS/PD12); no longer IC5.P12 (CAN2_RX/ETH_TXD0/I2C2_SMBA/I2S2_WS/SPI2_NSS/TIM1_BKIN/USART3_CK/USB_OTG_HS_ID/USB_OTG_HS_ULPI_D5/PB12)
- net RADIO_CS: now also IC5.D15 (DCMI_D1/TIM1_CH3/USART1_RX/USB_OTG_FS_ID/PA10); no longer IC5.P14 (DAC_EXTI9/FMC_D14/FMC_DA14/USART3_RX/PD9)
- net RADIO_GPIO0: now also IC5.N14 (ADC1_EXTI11/ADC2_EXTI11/ADC3_EXTI11/FMC_A16/FMC_CLE/I2C4_SMBA/QUADSPI_BK1_IO0/SAI2_SD_A/USART3_CTS/PD11); no longer IC5.N15 (FMC_D15/FMC_DA15/USART3_CK/PD10)
- net RADIO_GPIO2: now also U1.6 (SW1), W1.1
- net RADIO_GPIO3: now also W3.1, U1.4 (SW2)
- net RADIO_IRQ: now also IC5.N15 (FMC_D15/FMC_DA15/USART3_CK/PD10); no longer IC5.N14 (ADC1_EXTI11/ADC2_EXTI11/ADC3_EXTI11/FMC_A16/FMC_CLE/I2C4_SMBA/QUADSPI_BK1_IO0/SAI2_SD_A/USART3_CTS/PD11)
- net RADIO_SDN: now also IC5.P14 (DAC_EXTI9/FMC_D14/FMC_DA14/USART3_RX/PD9); no longer IC5.N13 (FMC_A17/FMC_ALE/I2C4_SCL/LPTIM1_IN1/QUADSPI_BK1_IO1/SAI2_FS_A/TIM4_CH1/USART3_RTS/PD12)
- net SPI_MISO: now also IC5.C14 (PI2/DCMI_D9/FMC_D26/SPI2_MISO/TIM8_CH4); no longer IC5.R14 (SPI2_MISO/TIM12_CH1/TIM1_CH2N/TIM8_CH2N/USART3_RTS/USB_OTG_HS_DM/PB14)
- net SPI_MOSI: now also IC5.C13 (PI3/DCMI_D10/FMC_D27/I2S2_SD/SPI2_MOSI/TIM8_ETR); no longer IC5.R15 (I2S2_SD/RTC_REFIN/SPI2_MOSI/TIM12_CH2/TIM1_CH3N/TIM8_CH3N/USB_OTG_HS_DP/PB15)
- net SPI_SCK: now also IC5.D14 (PI1/DCMI_D8/FMC_D25/I2S2_CK/SPI2_SCK/TIM8_BKIN2); no longer IC5.P13 (CAN2_TX/ETH_TXD1/I2S2_CK/SPI2_SCK/TIM1_CH1N/USART3_CTS/USB_OTG_HS_ULPI_D6/USB_OTG_HS_VBUS/PB13)
- net USB_D+: now also IC5.R15 (I2S2_SD/RTC_REFIN/SPI2_MOSI/TIM12_CH2/TIM1_CH3N/TIM8_CH3N/USB_OTG_HS_DP/PB15); no longer IC5.B15 (CAN1_TX/SAI2_FS_B/TIM1_ETR/USART1_RTS/USB_OTG_FS_DP/PA12)
- net USB_D-: now also IC5.R14 (SPI2_MISO/TIM12_CH1/TIM1_CH2N/TIM8_CH2N/USART3_RTS/USB_OTG_HS_DM/PB14); no longer IC5.C15 (ADC1_EXTI11/ADC2_EXTI11/ADC3_EXTI11/CAN1_RX/TIM1_CH4/USART1_CTS/USB_OTG_FS_DM/PA11)
- net USB_VUSB: now also IC5.P13 (CAN2_TX/ETH_TXD1/I2S2_CK/SPI2_SCK/TIM1_CH1N/USART3_CTS/USB_OTG_HS_ULPI_D6/USB_OTG_HS_VBUS/PB13); no longer IC5.E15 (DAC_EXTI9/DCMI_D0/I2C3_SMBA/I2S2_CK/SPI2_SCK/TIM1_CH2/USART1_TX/USB_OTG_FS_VBUS/PA9)
- net VDDA: now also P1.5 (P5)
- net V_BOOST: now also P3.4 (ID)
- net CAM_GPIO2: now reaches IC5.A2 (ETH_TXD3/FMC_A23/QUADSPI_BK1_IO2/SAI1_MCLK_A/SPI4_SCK/SYS_TRACECLK/PE2)
- net CAM_GPIO2: now also P1.8 (P8)
- net CAM_GPIO1: now reaches IC5.A3 (DCMI_D3/FMC_NBL1/LPTIM1_IN2/UART8_TX/PE1)
- net CAM_GPIO1: now also P1.13 (P13)
- net CAM_GPIO0: now reaches IC5.A4 (DCMI_D2/FMC_NBL0/LPTIM1_ETR/SAI2_MCLK_A/TIM4_ETR/UART8_RX/PE0)
- net CAM_GPIO0: now also P1.15 (P15)
- net +IO: now reaches IC5.B10 (PG10/DCMI_D2/FMC_NE3/SAI2_SD_B)
- net +IO: now also IC5.B9 (PG11/ADC1_EXTI11/ADC2_EXTI11/ADC3_EXTI11/DCMI_D3/ETH_TX_EN/SPDIFRX_IN0), IC5.C10 (PG9/DAC_EXTI9/DCMI_VSYNC/FMC_NCE3/FMC_NE2/QUADSPI_BK2_IO2/SAI2_FS_B/SPDIFRX_IN3/USART6_RX), IC6.20 (VCC_IO), R38.2
- net at IC6.1 (RF_IN): now also P6.1; no longer W3.1
- net at IC4.16 (XOUT): no longer C17.2
- net at IC4.4 (TX), L3.1: now also C19.2; no longer C19.1
- net at L4.2: now also C19.1; no longer C19.2
- net at C24.2: now also P4.1
- net at C51.2: now also U1.3 (IN2)
- removed net USB_ID: IC5.D15 (DCMI_D1/TIM1_CH3/USART1_RX/USB_OTG_FS_ID/PA10), P3.4 (ID), R31.2
- new net: L4.1, R37.1, U1.1 (IN1)
- new net: R37.2, U1.5 (OUT), U2.1 (IN)
- new net: C24.1, U2.2 (OUT)
- new net: D10.1 (K), P7.15 (P15)
- new net: D10.2 (A), R34.2
- new net OV2640_AVDD: C21.1, P7.5 (P5), U3.17 (AVDD)
- new net OV2640_D2: P7.19 (P19), U3.2 (Y2)
- new net OV2640_D3: P7.24 (P24), U3.19 (Y3)
- new net OV2640_D4: P7.23 (P23), U3.13 (Y4)
- new net OV2640_D5: P7.22 (P22), U3.23 (Y5)
- new net OV2640_D6: P7.4 (P4), U3.3 (Y6)
- new net OV2640_D7: P7.17 (P17), U3.24 (Y7)
- new net OV2640_D8: P7.10 (P10), U3.4 (Y8)
- new net OV2640_D9: P7.18 (P18), U3.1 (Y9)
- new net OV2640_DOVDD: P7.9 (P9), U3.22 (DOVDD)
- new net OV2640_DVDD: P7.7 (P7), U3.20 (DVDD)
- new net OV2640_HREF: P7.11 (P11), U3.10 (HREF)
- new net OV2640_PCLK: P7.20 (P20), U3.21 (PCLK)
- new net OV2640_PWDN: P7.8 (P8), U3.9 (PWDN)
- new net OV2640_RESET: P7.6 (P6), U3.7 (RESET)
- new net OV2640_SCL: IC9.4 (SCK), P7.14 (P14), U3.14 (SIO_C)
- new net OV2640_SDA: IC9.3 (SDI), P7.12 (P12), U3.15 (SIO_D)
- new net OV2640_VSYNC: P7.16 (P16), U3.12 (VSYNC)
- new net OV2640_XCLK: P7.21 (P21), U3.5 (XCLK)
Other:
- note added: "2m Transceiver"
- note added: "ADP controls the supply\nvoltage for the camera\nand the GPS. Both need\na clean voltage."
- note added: "Battery"
- note added: "Battery connection\npads"
- note added: "Camera edge connector and daugther board (camera + additional BME280)"
- note added: "Clock CTRL may be used to modulate\nthe Si4464. It may also influence the\nclock of the STM32 but only slightly."
- note added: "Connectors"
- note added: "Debug"
- note added: "Duplicate BME280 on the camera daughter board.\nIC9 may be used instead of IC8 because it is more\nfar away from heat sources. It may measure the\ntemperature and humidity more accurately.\nNote: IC8 and IC9 have different addresses."
- note added: "If you don't want to use the receiver,\nyou may fit R37 and remove U1."
- note added: "LCN-120 is ideal for\n2m band (144-148MHz)"
- note added: "Microcontroller must\nfeed VCC_IO unless\nR38 is fitted."
- note added: "Power"
- note added: "Programming"
- note added: "Put jumper on Pins 10 and 11\nin order to connect the battery\nto the actual circuit. So you\ndon't have to desolder the\nbattery everytime."
- note added: "Sensors and GPS"
- note added: "Solar"
- note added: "Solar cells must be\nconnected to pad W7\nand W10."
- note added: "Solar left-to-right\ninterconnection"
- note added: "The battery can be charged by USB.\nThe USB supply is not connected directly\nto the SPV1040 while the input voltage\nmust not exceed by 4.1V."
- note added: "USB only work with USB hosts like computer.\nThe USB ID pin used to switch VCC from 1.8V to 3.3V\nUSB Slaves like USB Sticks do not work, because\nUSB ID pin is not connected to STM32."
- note added: "V_BOOST is pulled down by STM32 or by USB Host.\nWhen V_BOOST is pulled down the TPS62260 will\nswitch to 3.0V. This is necessary for USB commu-\nnication and to get more power out of the Si4464.\nV_BOOST must not be pulled high because the\nTPS62260 will fail."
- note added: "Voltage can be\nmeasured by IC7"
- note added: "not fitted"
- moved on the sheet: C1, C10, C11, C12, C13, C14, C15, C16, C18, C19, C2, C20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

Commit message: Added new LDO for GPS Implemented constant voltage for LEDs Replaced MicroUSB THT connector with SMD connector Replaced LPF
Parts:
- removed C51: 470p, stm32f7:C_0402, symbol C
- removed D5: red, stm32f7:LED_0603, symbol LED
- removed D6: green, stm32f7:LED_0603, symbol LED
- removed IC8: BME280, stm32f7:BME280, symbol BME280
- removed L7: 56n, stm32f7:R_0402, symbol INDUCTOR
- removed R13: 100k, stm32f7:R_0402, symbol R
- removed R15: 1k5, stm32f7:R_0402, symbol R
- removed R16: 330R, stm32f7:R_0402, symbol R
- removed R37, R38: 0R, stm32f7:R_0402, symbol R
- removed U1: AS-213, stm32f7:SC-70-6, symbol RF_SWITCH
- removed U2: LFCN-120, stm32f7:FV1206, symbol LPF
- removed W3: Testpad, stm32f7:Testpad, symbol TEST_1P
- added C25, C27: 470p, stm32f7:C_0402, symbol C
- added C26: 22p, stm32f7:C_0402, symbol C
- added IC8: LDLN015PU30R, Housings_DFN_QFN:DFN-6-1EP_2x2mm_Pitch0.5mm, symbol LDLN015
- added L5: 82n, stm32f7:C_0805, symbol INDUCTOR
- added L6: 56n, stm32f7:C_0805, symbol INDUCTOR
- C24: value 470p -> 22p
- C50: value 470p -> 22u; footprint stm32f7:C_0402 -> stm32f7:C_0805
- D1: value green -> yellow
- D2: value green -> blue
- D4: value green -> red
- L3, L4: footprint stm32f7:R_0603 -> stm32f7:C_0805
- P3: value USB_OTG -> ZX62-B-5PA(33); footprint stm32f7:USB_Micro-B -> stm32f7:USB_Micro-B_SMD
- R21: value 1k5 -> 1k
- W1: footprint stm32f7:Testpad -> stm32f7:PAD_3x1.5
Connections:
- net +1V8: no longer C29.1, R10.1, R11.1, R12.1, R34.1, R9.1
- net +3V3: now also IC7.10 (VDD), R10.1, R11.1, R12.1, R9.1; no longer C20.1, C22.1, D7.2 (A), IC6.19 (VCC)
- net GND: now also C24.2, C50.2, C26.2, IC8.4 (GND), IC8.7 (THERM); no longer C50.1
- net GPS_EN: now also IC5.B14 (DCMI_D8/I2S3_CK/QUADSPI_BK1_IO1/SDMMC1_D2/SPI3_SCK/UART4_TX/USART3_TX/PC10), IC8.3 (EN); no longer IC3.1 (EN1), IC5.J2 (PF3/ADC3_IN9/FMC_A3)
- net OV2640_AVDD: now also R34.1
- net at IC4.2 (RX+): no longer C50.2
- net at L4.1: now also C24.1, C25.1, L5.2
- net at P4.1: now also W1.1, C27.2, L6.1; no longer C24.2
- removed net +IO: IC5.B10 (PG10/DCMI_D2/FMC_NE3/SAI2_SD_B), IC5.B9 (PG11/ADC1_EXTI11/ADC2_EXTI11/ADC3_EXTI11/DCMI_D3/ETH_TX_EN/SPDIFRX_IN0), IC5.C10 (PG9/DAC_EXTI9/DCMI_VSYNC/FMC_NCE3/FMC_NE2/QUADSPI_BK2_IO2/SAI2_FS_B/SPDIFRX_IN3/USART6_RX), IC6.20 (VCC_IO)
- net PAC_ALERT: no longer names the net of IC5.N13 (FMC_A17/FMC_ALE/I2C4_SCL/LPTIM1_IN1/QUADSPI_BK1_IO1/SAI2_FS_A/TIM4_CH1/USART3_RTS/PD12)
- net PAC_ALERT: no longer IC7.7 (ALERT)
- net RADIO_GPIO2: no longer names the net of IC4.19 (GPIO2)
- net RADIO_GPIO2: no longer W1.1
- net RADIO_GPIO3: no longer names the net of IC4.20 (GPIO3)
- net SENSE_BAT- renamed VDD
- net VDD: now also C29.1, C50.1, IC3.1 (EN1), IC8.1 (IN); no longer IC7.10 (VDD)
- new net: C25.2, C26.1, C27.1, L5.1, L6.2
- new net VCC_GPS: C20.1, C22.1, D7.2 (A), IC6.19 (VCC), IC6.20 (VCC_IO), IC8.6 (OUT)
Other:
- note added: "+BATT Directly connected to battery\n+SOL Solar network\nVDD Connected to battery through sense resistor\n+1V8 Main power supply for STM32 and transmitter\n+3V3 LED and PAC1720 power supply\n+VDDA Analog power supply for camera\n+1V35 Core power supply for camery (actually 1.8V)"
- note added: "GPS"
- note removed: "If you don't want to use the receiver,\nyou may fit R37 and remove U1."
- note removed: "LCN-120 is ideal for\n2m band (144-148MHz)"
- note removed: "Microcontroller must\nfeed VCC_IO unless\nR38 is fitted."
- note removed: "Sensors and GPS"
- note removed: "not fitted"
- moved on the sheet: C20, C22, C23, C48, C49, D10, D7, IC6, P4, P6, R19, R20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

Commit message: Moving parts around
Connections:
- net +1V8: now also IC9.5 (SDO)
- net +SOL: now also F1.2; no longer D8.1 (K)
- net GND: no longer IC9.5 (SDO)
- net GPS_RESET: now also IC5.A9 (I2S2_WS/SPI1_MISO/SPI2_NSS/SPI3_MISO/SYS_JTRST/TIM3_CH1/PB4); no longer IC5.A11 (FMC_NE1/SPDIFRX_IN0/USART2_CK/PD7)
- net GPS_TIMEPULSE: now also IC5.A11 (FMC_NE1/SPDIFRX_IN0/USART2_CK/PD7); no longer IC5.A9 (I2S2_WS/SPI1_MISO/SPI2_NSS/SPI3_MISO/SYS_JTRST/TIM3_CH1/PB4)
- net USB_VUSB: now also D9.2 (A); no longer F1.2
- net at F1.1: now also D8.1 (K); no longer D9.2 (A)
Other:
- moved on the sheet: D8, D9, F1
Changed lines of the file:
@@
 L DIODE D9
 U 1 1 57ACA15E
-P 18550 11200
-F 0 "D9" H 18550 11350 50  0000 C CNN
-F 1 "DIODE" H 18550 11025 50  0000 C CNN
-F 2 "Diodes_SMD:MELF_Standard" H 18550 11200 50  0001 C CNN
-F 3 "" H 18550 11200 50  0000 C CNN
-	1    18550 11200
+P 18700 11200
+F 0 "D9" H 18700 11350 50  0000 C CNN
+F 1 "DIODE" H 18700 11025 50  0000 C CNN
+F 2 "Diodes_SMD:MELF_Standard" H 18700 11200 50  0001 C CNN
+F 3 "" H 18700 11200 50  0000 C CNN
+	1    18700 11200
 	1    0    0    -1
 $EndComp
@@
 L DIODE D8
 U 1 1 57ACB163
-P 18050 11200
-F 0 "D8" H 18050 11350 50  0000 C CNN
-F 1 "DIODE" H 18050 11025 50  0000 C CNN
-F 2 "Diodes_SMD:MELF_Standard" H 18050 11200 50  0001 C CNN
-F 3 "" H 18050 11200 50  0000 C CNN
-	1    18050 11200
+P 18200 11200
+F 0 "D8" H 18200 11350 50  0000 C CNN
+F 1 "DIODE" H 18200 11025 50  0000 C CNN
+F 2 "Diodes_SMD:MELF_Standard" H 18200 11200 50  0001 C CNN
+F 3 "" H 18200 11200 50  0000 C CNN
+	1    18200 11200
 	1    0    0    -1
 $EndComp
@@
 L F_Small F1
 U 1 1 57AE057D
-P 19000 11450
-F 0 "F1" H 18960 11510 50  0000 L CNN
-F 1 "500mA" H 18880 11390 50  0000 L CNN
-F 2 "Fuse_Holders_and_Fuses:Fuse_SMD1206_Reflow" H 19000 11450 50  0001 C CNN
-F 3 "" H 19000 11450 50  0000 C CNN
-	1    19000 11450
-	0    1    1    0
+P 17750 11200
+F 0 "F1" H 17710 11260 50  0000 L CNN
+F 1 "500mA" H 17630 11140 50  0000 L CNN
+F 2 "Fuse_Holders_and_Fuses:Fuse_SMD1206_Reflow" H 17750 11200 50  0001 C CNN
+F 3 "" H 17750 11200 50  0000 C CNN
+	1    17750 11200
+	-1   0    0    1
 $EndComp
 Text Label 18500 12100 0    60   ~ 0
@@
 	0    -1   -1   0
 $EndComp
-Text Label 20600 7700 2    60   ~ 0
+Text Label 20600 4000 2    60   ~ 0
 GPS_RESET
 $Comp
@@
 Text Label 20600 2200 2    60   ~ 0
 ADC_VSOL
-Text Label 20600 4000 2    60   ~ 0
+Text Label 20600 7700 2    60   ~ 0
 GPS_TIMEPULSE
 $Comp
@@
 OV2640_SDA
 $Comp
-L GND #PWR0101
-U 1 1 587343EA
-P 15700 13000
-F 0 "#PWR0101" H 15700 12750 50  0001 C CNN
-F 1 "GND" H 15700 12850 50  0000 C CNN
-F 2 "" H 15700 13000 50  0000 C CNN
-F 3 "" H 15700 13000 50  0000 C CNN
-	1    15700 13000
-	1    0    0    -1
-$EndComp
-$Comp
-L +1V8 #PWR0102
+L +1V8 #PWR0101
 U 1 1 5873311D
 P 15700 12250
-F 0 "#PWR0102" H 15700 12100 50  0001 C CNN
+F 0 "#PWR0101" H 15700 12100 50  0001 C CNN
 F 1 "+1V8" H 15700 12390 50  0000 C CNN
 F 2 "" H 15700 12250 50  0000 C CNN
@@
 $EndComp
 $Comp
-L +1V8 #PWR0103
+L +1V8 #PWR0102
 U 1 1 58733123
 P 14400 12250
-F 0 "#PWR0103" H 14400 12100 50  0001 C CNN
+F 0 "#PWR0102" H 14400 12100 50  0001 C CNN
 F 1 "+1V8" H 14400 12390 50  0000 C CNN
 F 2 "" H 14400 12250 50  0000 C CNN
@@
 $EndComp
 $Comp
-L +1V8 #PWR0104
+L +1V8 #PWR0103
 U 1 1 587369D9
 P 12150 12300
-F 0 "#PWR0104" H 12150 12150 50  0001 C CNN
+F 0 "#PWR0103" H 12150 12150 50  0001 C CNN
 F 1 "+1V8" H 12150 12440 50  0000 C CNN
 F 2 "" H 12150 12300 50  0000 C CNN
@@
 $EndComp
 $Comp
-L +1V8 #PWR0105
+L +1V8 #PWR0104
 U 1 1 58737733
 P 12150 14100
-F 0 "#PWR0105" H 12150 13950 50  0001 C CNN
+F 0 "#PWR0104" H 12150 13950 50  0001 C CNN
 F 1 "+1V8" H 12150 14240 50  0000 C CNN
 F 2 "" H 12150 14100 50  0000 C CNN
@@
 $EndComp
 $Comp
-L GND #PWR0106
+L GND #PWR0105
 U 1 1 58731CFB
 P 11600 13900
-F 0 "#PWR0106" H 11600 13650 50  0001 C CNN
+F 0 "#PWR0105" H 11600 13650 50  0001 C CNN
 F 1 "GND" H 11600 13750 50  0000 C CNN
 F 2 "" H 11600 13900 50  0000 C CNN
@@
 $EndComp
 $Comp
-L GND #PWR0107
+L GND #PWR0106
 U 1 1 587BEC6D
 P 20700 4800
-F 0 "#PWR0107" H 20700 4550 50  0001 C CNN
+F 0 "#PWR0106" H 20700 4550 50  0001 C CNN
 F 1 "GND" H 20700 4650 50  0000 C CNN
 F 2 "" H 20700 4800 50  0000 C CNN
@@
 	18500 12100 19100 12100
 Wire Wire Line
-	19000 11350 19000 11200
-Wire Wire Line
-	19000 11550 19000 11800
+	19000 11200 19000 11800
 Wire Wire Line
 	2100 10150 2100 10100
@@
 Wire Wire Line
 	4800 9150 7600 9150
-Wire Wire Line
-	17750 11200 17850 11200
 Wire Wire Line
 	18400 11800 19100 11800
@@
 	15700 12400 15600 12400
 Wire Wire Line
-	15700 12250 15700 12400
+	15700 12250 15700 12800
 Connection ~ 14700 12800
 Wire Wire Line
@@
 Wire Wire Line
 	14800 12800 14700 12800
-Wire Wire Line
-	15700 13000 15700 12800
 Wire Wire Line
 	12150 12500 12150 12300
@@
 GPS
 $Comp
-L +SOL #PWR0108
+L +SOL #PWR0107
 U 1 1 5882D1D5
-P 17750 11200
-F 0 "#PWR0108" H 17750 11050 50  0001 C CNN
-F 1 "+SOL" H 17750 11340 50  0000 C CNN
-F 2 "" H 17750 11200 50  0000 C CNN
-F 3 "" H 17750 11200 50  0000 C CNN
-	1    17750 11200
+P 17500 11200
+F 0 "#PWR0107" H 17500 11050 50  0001 C CNN
+F 1 "+SOL" H 17500 11340 50  0000 C CNN
+F 2 "" H 17500 11200 50  0000 C CNN
+F 3 "" H 17500 11200 50  0000 C CNN
+	1    17500 11200
 	0    -1   -1   0
 $EndComp
 Wire Wire Line
-	19000 11200 18750 11200
-Wire Wire Line
-	18350 11200 18250 11200
+	19000 11200 18900 11200
+Wire Wire Line
+	18500 11200 18400 11200
 Wire Notes Line
 	19550 13350 17550 13350
@@
 Connection ~ 4050 2900
 $Comp
-L +3V3 #PWR0109
+L +3V3 #PWR0108
 U 1 1 58C07E50
 P 20900 8500
-F 0 "#PWR0109" H 20900 8350 50  0001 C CNN
+F 0 "#PWR0108" H 20900 8350 50  0001 C CNN
 F 1 "+3V3" H 20900 8640 50  0000 C CNN
 F 2 "" H 20900 8500 50  0000 C CNN
@@
 $EndComp
 $Comp
-L +3V3 #PWR0110
+L +3V3 #PWR0109
 U 1 1 58C08B6E
 P 21200 8500
-F 0 "#PWR0110" H 21200 8350 50  0001 C CNN
+F 0 "#PWR0109" H 21200 8350 50  0001 C CNN
 F 1 "+3V3" H 21200 8640 50  0000 C CNN
 F 2 "" H 21200 8500 50  0000 C CNN
@@
 $EndComp
 $Comp
-L +3V3 #PWR0111
+L +3V3 #PWR0110
 U 1 1 58C08D2C
 P 20950 2600
-F 0 "#PWR0111" H 20950 2450 50  0001 C CNN
+F 0 "#PWR0110" H 20950 2450 50  0001 C CNN
 F 1 "+3V3" H 20950 2740 50  0000 C CNN
 F 2 "" H 20950 2600 50  0000 C CNN
@@
 $EndComp
 $Comp
-L +3V3 #PWR0112
+L +3V3 #PWR0111
 U 1 1 58C09D29
 P 21250 2600
-F 0 "#PWR0112" H 21250 2450 50  0001 C CNN
+F 0 "#PWR0111" H 21250 2450 50  0001 C CNN
 F 1 "+3V3" H 21250 2740 50  0000 C CNN
 F 2 "" H 21250 2600 50  0000 C CNN
@@
 Connection ~ 4350 2900
 $Comp
-L VDD #PWR0113
+L VDD #PWR0112
 U 1 1 58C1366F
 P 7250 9050
-F 0 "#PWR0113" H 7250 8900 50  0001 C CNN
+F 0 "#PWR0112" H 7250 8900 50  0001 C CNN
 F 1 "VDD" H 7250 9200 50  0000 C CNN
 F 2 "" H 7250 9050 50  0000 C CNN
@@
 $EndComp
 $Comp
-L VDD #PWR0114
+L VDD #PWR0113
 U 1 1 58C14161
 P 6950 6500
-F 0 "#PWR0114" H 6950 6350 50  0001 C CNN
+F 0 "#PWR0113" H 6950 6350 50  0001 C CNN
 F 1 "VDD" H 6950 6650 50  0000 C CNN
 F 2 "" H 6950 6500 50  0000 C CNN
@@
 Connection ~ 6950 6600
 $Comp
-L +3V3 #PWR0115
+L +3V3 #PWR0114
 U 1 1 58C1656D
 P 7350 10500
-F 0 "#PWR0115" H 7350 10350 50  0001 C CNN
+F 0 "#PWR0114" H 7350 10350 50  0001 C CNN
 F 1 "+3V3" H 7350 10640 50  0000 C CNN
 F 2 "" H 7350 10500 50  0000 C CNN
@@
 $EndComp
 $Comp
-L GND #PWR0116
+L GND #PWR0115
 U 1 1 58C251B3
 P 5600 14850
-F 0 "#PWR0116" H 5600 14600 50  0001 C CNN
+F 0 "#PWR0115" H 5600 14600 50  0001 C CNN
 F 1 "GND" H 5600 14700 50  0000 C CNN
 F 2 "" H 5600 14850 50  0000 C CNN
@@
 $EndComp
 $Comp
-L GND #PWR0117
+L GND #PWR0116
 U 1 1 58C2535A
 P 6400 14850
-F 0 "#PWR0117" H 6400 14600 50  0001 C CNN
+F 0 "#PWR0116" H 6400 14600 50  0001 C CNN
 F 1 "GND" H 6400 14700 50  0000 C CNN
 F 2 "" H 6400 14850 50  0000 C CNN
@@
 	4500 3000 4500 3200
 $Comp
-L GND #PWR0118
+L GND #PWR0117
 U 1 1 58C33013
 P 4500 3200
-F 0 "#PWR0118" H 4500 2950 50  0001 C CNN
+F 0 "#PWR0117" H 4500 2950 50  0001 C CNN
 F 1 "GND" H 4500 3050 50  0000 C CNN
 F 2 "" H 4500 3200 50  0000 C CNN
@@
 	5400 2900 5400 3250
 $Comp
-L VDD #PWR0119
+L VDD #PWR0118
 U 1 1 58C34563
 P 5650 2800
-F 0 "#PWR0119" H 5650 2650 50  0001 C CNN
+F 0 "#PWR0118" H 5650 2650 50  0001 C CNN
 F 1 "VDD" H 5650 2950 50  0000 C CNN
 F 2 "" H 5650 2800 50  0000 C CNN
@@
 $EndComp
 $Comp
-L GND #PWR0120
+L GND #PWR0119
 U 1 1 58C3503A
 P 5400 3600
-F 0 "#PWR0120" H 5400 3350 50  0001 C CNN
+F 0 "#PWR0119" H 5400 3350 50  0001 C CNN
 F 1 "GND" H 5400 3450 50  0000 C CNN
 F 2 "" H 5400 3600 50  0000 C CNN
@@
 $EndComp
 $Comp
-L GND #PWR0121
+L GND #PWR0120
 U 1 1 58C35A79
 P 5650 3600
-F 0 "#PWR0121" H 5650 3350 50  0001 C CNN
+F 0 "#PWR0120" H 5650 3350 50  0001 C CNN
 F 1 "GND" H 5650 3450 50  0000 C CNN
 F 2 "" H 5650 3600 50  0000 C CNN
@@
 Text Notes 2200 7350 0    60   ~ 0
 +BATT Directly connected to battery\n+SOL Solar network\nVDD Connected to battery through sense resistor\n+1V8 Main power supply for STM32 and transmitter\n+3V3 LED and PAC1720 power supply\n+VDDA Analog power supply for camera\n+1V35 Core power supply for camery (actually 1.8V)
+Connection ~ 15700 12400
+Wire Wire Line
+	17500 11200 17650 11200
+Wire Wire Line
+	17850 11200 18000 11200
 $EndSCHEMATC
