File: hardware/pecanpico8.sch (KiCad schematic (older format))
At the start: 138 parts, among them IC1 SPV1040, IC2 TPS62260, IC3 ADP322ACPZ-115-R7, IC4 Si4464, IC5 STM32F745IGKx, IC6 EVA-7M, IC7 PAC1720, IC8 LDLN015PU30R, IC9 BME280, P1 CONN_02X13, P2 CONN_01X11, P3 ZX62-B-5PA(33), P4 IPX 2mm, P5 CONN_01X02, P6 IPX 2mm, P7 CONN_02X13, Q1 FDN306P, U3 uctronics OV2640, X1 KT2016K26000BCW18ZAS

Commit message: Replaced inductor for SPV1040, added production information, created GERBERs
Parts:
- added R13: N/A, stm32f7:R_0402, symbol R
- C1, C18, C19, C2, C24, C25, C26, C27, C3, C4, C7, C8, C9: Specs (none) -> 16V
- C10, C11, C12, C13, C14, C15, C16, C17, C20, C21, C22, C23, C29, C30, C31, C32, C33, C34, C35, C36, C37, C38, C39, C40, C41, C42, C43, C44, C45, C46, C47, C48, C49, C5, C50, C6: Specs (none) -> 10V
- C28: value ? -> 1u; Specs (none) -> 10V
- D8, D9: value DIODE -> RFN1L7STE25; Mouser (none) -> 755-RFN1L7STE25
- F1: value 500mA -> PMS1206-075; Mouser (none) -> 637-PMS1206-075; Specs (none) -> 750mA
- IC1: value SPV1040 -> SPV1040T; Mouser (none) -> 511-SPV1040T
- IC2: value TPS62260 -> TPS62260DRVR; Mouser (none) -> 595-TPS62260DRVR
- IC3: Mouser (none) -> 584-ADP322ACPZ-115R7
- IC4: value Si4464 -> Si4063-B1B-FM; Mouser (none) -> 634-SI4063-B1B-FM
- IC5: value STM32F745IGKx -> STM32F429IIH6; Mouser (none) -> 511-STM32F429IIH6
- IC6: Notes (none) -> get from uBlox directly
- IC7: value PAC1720 -> PAC1720-1-AIA-TR; Mouser (none) -> 579-PAC1720-1-AIA-TR
- IC8: value LDLN015PU30R -> LDLN015PU33R; Mouser (none) -> 511-LDLN015PU33R
- IC9: Mouser (none) -> 262-BME280
- L1: value 10u -> XAL4040-103; footprint stm32f7:LPS3015 -> stm32f7:XAL4040; Mouser (none) -> 994-XAL4040-103MEC
- L2: value 2u2 -> LPS3015-222; Mouser (none) -> 994-LPS3015-222MRC
- L3: Mouser (none) -> 994-0805LS-471XJLB
- L4, L6: Mouser (none) -> 994-0805CS-560XJLC
- L5: Mouser (none) -> 994-0805CS-820XJLC
- P1, P2, P5, P7, W1, W10, W11, W12, W13, W14, W15, W16, W17, W18, W19, W20, W21, W22, W23, W24, W26, W27, W6, W7, W8: Notes (none) -> do not assemble
- P3: Mouser (none) -> 798-ZX62-B-5PA33
- P4, P6: Mouser (none) -> 960-RECE20279001E01
- Q1: Mouser (none) -> 512-FDN306P
- R1, R14, R17, R2, R23, R24, R25, R26, R28, R3, R31, R32, R33, R35, R36, R4, R5, R6, R7, R8: Specs (none) -> 1%
- R10, R11, R12, R9: value 0R -> 1k5; Specs (none) -> 1%
- R18, R22: Mouser (none) -> 71-WSLP0603R1000FEA
- R19, R20: value 0R -> N/A; Notes (none) -> do not assemble
- R21: value 1k -> 1k5; Specs (none) -> 1%
- R29, R30: value ? -> 1k; Specs (none) -> 1%
- R34: value 0R -> 1k; Specs (none) -> 1%
- U3: Notes (none) -> Get here https://www.alibaba.com/product-detail/2-0-Mega-Pi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
- X1: Mouser (none) -> 581-KT2016K2BCW18ZAS
Connections:
- net GND: now also R13.2
- net SOL_SHORT_EN: now also R13.1
Other:
- note added: "If SOL_SHORT_EN is enabled, the\ncurrent of the solar cell can be\nmeasured by the PAC1720"
- moved on the sheet: D8, F1

Commit message: Fixed wrong comment
Other:
- note added: "Clock CTRL may be used to modulate\nthe Si4063. It may also influence the\nclock of the STM32 but only slightly."
- note removed: "Clock CTRL may be used to modulate\nthe Si4464. It may also influence the\nclock of the STM32 but only slightly."
Changed lines of the file:
@@
 USB only work with USB hosts like computer.\nThe USB ID pin used to switch VCC from 1.8V to 3.3V\nUSB Slaves like USB Sticks do not work, because\nUSB ID pin is not connected to STM32.
 Text Notes 6450 3550 0    60   ~ 0
-Clock CTRL may be used to modulate\nthe Si4464. It may also influence the\nclock of the STM32 but only slightly.
+Clock CTRL may be used to modulate\nthe Si4063. It may also influence the\nclock of the STM32 but only slightly.
 Text Notes 2400 10600 0    60   ~ 0
 Voltage can be\nmeasured by IC7
